File: kicad_files/athena.kicad_sch (KiCad schematic)
At the start: 245 parts, among them J1 SM04B-SRSS-TB(LF)(SN), J2 TYPE-C-31-M12, J3 SM04B-SRSS-TB(LF)(SN), J4 ARM JTAG, J5 EXTRA PINS, Q1 DTC123JKAT146, SW1 MX Switch, SW10 MX Switch, SW100 MX Switch, SW101 MX Switch, SW102 MX Switch, SW103 MX Switch, SW104 MX Switch, SW105 MX Switch, SW106 MX Switch, SW107 MX Switch, SW108 MX Switch, SW109 MX Switch, SW11 MX Switch, SW110 MX Switch, SW111 MX Switch, SW112 MX Switch, SW113 K2-1187SQ-A4SW-06, SW12 MX Switch, SW13 MX Switch, SW14 MX Switch, SW15 MX Switch, SW16 MX Switch, SW17 MX Switch, SW18 MX Switch, SW19 MX Switch, SW2 MX Switch, SW20 MX Switch, SW21 MX Switch, SW22 MX Switch, SW23 MX Switch, SW24 MX Switch, SW25 MX Switch, SW26 MX Switch, SW27 MX Switch, SW28 MX Switch, SW29 MX Switch, SW3 MX Switch, SW30 MX Switch, SW31 MX Switch, SW32 MX Switch, SW33 MX Switch, SW34 MX Switch, SW35 MX Switch, SW36 MX Switch, SW37 MX Switch, SW38 MX Switch, SW39 MX Switch, SW4 MX Switch, SW40 MX Switch, SW41 MX Switch, SW42 MX Switch, SW43 MX Switch, SW44 MX Switch, SW45 MX Switch, SW46 MX Switch, SW47 MX Switch, SW48 MX Switch, SW49 MX Switch, SW5 MX Switch, SW50 MX Switch, SW51 MX Switch, SW52 MX Switch, SW53 MX Switch, SW54 MX Switch, SW55 MX Switch, SW56 MX Switch, SW57 MX Switch, SW58 MX Switch, SW59 MX Switch, SW6 MX Switch, SW60 MX Switch, SW61 MX Switch, SW62 MX Switch, SW63 MX Switch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

Commit message: Acheron Setup port, joker topology
- Tolerances and constraints were updated to Acheron Setup's defaults
- New MCU "joker" topology
Parts:
- removed C13: 100n, Capacitor_SMD:C_0402_1005Metric, symbol Device:C_Small
- removed C14: 4.7u, Capacitor_SMD:C_0402_1005Metric, symbol Device:C_Small
- removed J4: ARM JTAG, acheron_Connectors:Conn_ARM_JTAG_SWD_6, symbol Connector_Generic:Conn_02x03_Odd_Even
- removed J5: EXTRA PINS, acheron_Connectors:PinHeader_1x5_P2.54mm_Vertical, symbol Connector_Generic:Conn_01x05
- removed R5: 1.5k, Resistor_SMD:R_0402_1005Metric, symbol Device:R_Small
- removed U3: STM32F072CBT6, acheron_Components:LQFP-48_7x7mm_P0.5mm, symbol acheronSymbols:STM32F072-LQFP48
- added C1, C10, C2: 100n, Capacitor_SMD:C_0402_1005Metric, symbol Device:C_Small
- added C11: 2.2u, Capacitor_SMD:C_0402_1005Metric, symbol Device:C_Small
- added C12: 4.7u, Capacitor_SMD:C_0402_1005Metric, symbol Device:C_Small
- added C19, C20, C21, C22, C23, C24, C25, C26, C27, C28, C29, C30, C31, C32, C33, C34, C35: 100n, Capacitor_SMD:C_0805_2012Metric, symbol Device:C_Small
- added C7: 10n, Capacitor_SMD:C_0402_1005Metric, symbol Device:C_Small
- added D100, D101, D102, D103, D104, D105, D106, D107, D108, D109, D110, D111, D95, D96, D97, D98, D99: WS2812C, acheron_Components:LED_WS2812B_5.0x5.0mm_P3.2mm, symbol LED:WS2812B
- added LED1, LED10, LED11, LED12, LED13, LED14, LED15, LED16, LED17, LED18, LED19, LED2, LED20, LED21, LED22, LED23, LED24, LED25, LED26, LED27, LED28, LED29, LED3, LED30, LED31, LED32, LED33, LED34, LED35, LED36, LED37, LED38, LED39, LED4, LED40, LED41, LED42, LED43, LED44, LED5, LED6, LED7, LED8, LED9: LED, acheron_Components:LED_THT_2.54mm, symbol acheron_Symbols:LED
- added M1, M2: USB removal mousebite, athena_library:usbc_removal_mousebite_0.5mm, symbol Mechanical:MountingHole
- added M3, M4: USB removal mousebite, athena_library:usbc_removal_mousebite_1mm, symbol Mechanical:MountingHole
- added Q1: AO3401A, Package_TO_SOT_SMD:SOT-23, symbol Transistor_FET:AO3401A
- added R1, R2, R3: 1.5k, Resistor_SMD:R_0402_1005Metric, symbol Device:R_Small
- added R10, R11, R12, R13, R14, R15, R16, R17, R18, R19, R20, R21, R22, R23, R24, R25, R26, R27, R28, R29, R30, R31, R32, R33, R34, R35, R36, R37, R38, R39, R40, R41, R42, R8, R9: 470, Resistor_SMD:R_0805_2012Metric, symbol Device:R_Small
- added R6: 10k, Resistor_SMD:R_0805_2012Metric, symbol Device:R_Small
- added R7: 100, Resistor_SMD:R_0805_2012Metric, symbol Device:R_Small
- added U1: BL24C256A-SFRC, acheron_Components:TSSOP-8_4.4x3mm_P0.65mm, symbol Memory_EEPROM:24LC256
- added U2: STM32F411CEU6, acheron_Components:STM_UFQFPN-48_LQFP-48-1EP_7x7mm_P0.5mm_HandSoldering_ThermalReliefs, symbol acheron_Symbols:STM32F411-48
- added X1: ARM JTAG, acheron_Connectors:PinHeader_2x5_P2.54mm_Vertical_Staggered, symbol Connector_Generic:Conn_02x05_Odd_Even
- added Y1: 7325-0800A2010-00, acheron_Components:Crystal_SMD_3225-4Pin_3.2x2.5mm, symbol Device:Crystal_GND24
- C3, C4: Specification MLCC 10V -> MLCC 10V or more
- C5: value 100n -> 4.7u; Specification MLCC 10V -> MLCC 10V or more
- C6: value 4.7u -> 1u; Specification MLCC 10V -> MLCC 10V or more
- C8: value 1u -> 16p; Specification MLCC 10V -> (none)
- C9: value 10n -> 16p; Specification MLCC 10V -> (none)
- R4: value 1.5k -> 0R; footprint Resistor_SMD:R_0402_1005Metric -> Resistor_SMD:R_0805_2012Metric; Package R0402 -> R0805
- renumbered C1 to C13, C2 to C14, C7 to C15, C10 to C16, C11 to C17, C12 to C18, Q1 to Q2, R2 to R43, R3 to R44, R6 to R45, R7 to R46, R8 to R47, R9 to R48, R10 to R49, R1 to R5, U1 to U3, U2 to U4, U4 to U5
Connections:
- net 3V3: now also C4.2, C6.1, C1.2, C10.2, C12.2, C2.1, C7.1, R1.1, R2.1, R3.1, U1.8 (VCC), U2.1 (VBAT), U2.24 (VDD), U2.36 (VDD), U2.48 (VDD), U2.9 (VDDA/VREF+), X1.7 (Pin_7), X1.8 (Pin_8); no longer C4.1, C6.2, C8.1, C9.1, R4.1
- net 5V: now also F1.1, R4.1, C19.1, C20.2, C21.1, C22.1, C23.1, C24.1, C25.1, C26.1, C27.1, C28.1, C29.1, C30.1, C31.1, C32.1, C33.1, C34.1, C35.1, D100.1 (VDD), D101.1 (VDD), D102.1 (VDD), D103.1 (VDD), D104.1 (VDD), D105.1 (VDD), D106.1 (VDD), D107.1 (VDD), D108.1 (VDD), D109.1 (VDD), D110.1 (VDD), D111.1 (VDD), D95.1 (VDD), D96.1 (VDD), D97.1 (VDD), D98.1 (VDD), D99.1 (VDD), Q1.2 (S), R6.2; no longer F1.2
- net BOOT0: now also U2.44 (BOOT0), X1.5 (Pin_5)
- net D+: now also U4.3 (I/O2), R3.2, U2.33 (PA12); no longer U4.1 (I/O1)
- net D-: now also U4.1 (I/O1), U2.32 (PA11); no longer U4.3 (I/O2)
- net DBUS+: now also U4.4 (I/O2); no longer U4.6 (I/O1)
- net DBUS-: now also U4.6 (I/O1); no longer U4.4 (I/O2)
- net GND: now also C4.1, C6.2, C1.1, C10.1, C11.1, C12.1, C19.2, C2.2, C20.1, C21.2, C22.2, C23.2, C24.2, C25.2, C26.2, C27.2, C28.2, C29.2, C30.2, C31.2, C32.2, C33.2, C34.2, C35.2, C7.2, D100.3 (VSS), D101.3 (VSS), D102.3 (VSS), D103.3 (VSS), D104.3 (VSS), D105.3 (VSS), D106.3 (VSS), D107.3 (VSS), D108.3 (VSS), D109.3 (VSS), D110.3 (VSS), D111.3 (VSS), D95.3 (VSS), D96.3 (VSS), D97.3 (VSS), D98.3 (VSS), D99.3 (VSS), LED1.K, LED10.K, LED11.K, LED12.K, LED13.K, LED14.K, LED15.K, LED16.K, LED17.K, LED18.K, LED19.K, LED2.K, LED20.K, LED21.K, LED22.K, LED23.K, LED24.K, LED25.K, LED26.K, LED27.K, LED28.K, LED29.K, LED3.K, LED30.K, LED31.K, LED32.K, LED33.K, LED34.K, LED35.K, LED36.K, LED37.K, LED38.K, LED39.K, LED4.K, LED40.K, LED41.K, LED42.K, LED43.K, LED44.K, LED5.K, LED6.K, LED7.K, LED8.K, LED9.K, U1.1 (A0), U1.2 (A1), U1.3 (A2), U1.4 (GND), U1.7 (WP), U2.23 (VSS), U2.35 (VSS), U2.47 (VSS), U2.8 (VSSA), X1.10 (Pin_10), X1.3 (Pin_3), X1.4 (Pin_4), Y1.2, Y1.4; no longer C4.2, C6.1
- net NRST: now also U2.7 (NRST), X1.9 (Pin_9)
- net RGB_3V3: now also U2.28 (PB15)
- net SCL: now also R2.2, U1.6 (SCL), U2.42 (PB6)
- net SDA: now also R1.2, U1.5 (SDA), U2.43 (PB7); no longer R4.2
- net SWCLK: now also U2.37 (PA14), X1.2 (Pin_2)
- net SWDIO: now also U2.34 (PA13), X1.1 (Pin_1)
- net VBUS: now also F1.2; no longer F1.1
- new net: C11.2, U2.22 (VCAP_1)
- new net: D110.2 (DOUT), D111.4 (DIN)
- new net: D109.2 (DOUT), D110.4 (DIN)
- new net: D103.2 (DOUT), D104.4 (DIN)
- new net: D102.2 (DOUT), D103.4 (DIN)
- new net: LED5.A, LED6.A, R11.1
- new net: LED12.A, R15.2
- new net: Q1.3 (D), R10.1, R11.2, R12.2, R13.1, R14.1, R15.1, R16.1, R17.1, R18.1, R19.1, R20.1, R21.1, R22.1, R23.1, R24.1, R25.1, R26.1, R27.1, R28.1, R29.1, R30.1, R31.1, R32.1, R33.1, R34.1, R35.1, R36.1, R37.1, R38.1, R39.1, R40.1, R41.1, R42.1, R8.1, R9.1
- new net: LED26.A, R25.2
- new net: LED18.A, LED19.A, R19.2
- new net: LED44.A, R42.2
- new net: LED28.A, R27.2
- new net: LED16.A, LED17.A, R18.2
- new net: LED30.A, R29.2
- new net: LED7.A, LED8.A, R12.1
- new net: LED10.A, LED9.A, R13.2
- new net: LED1.A, R8.2
- new net: LED43.A, R41.2
- new net: LED36.A, R35.2
- new net: LED40.A, LED41.A, R39.2
- new net: LED27.A, R26.2
- new net: LED34.A, R33.2
- new net: LED22.A, R21.2
- new net: LED3.A, LED4.A, R10.2
- new net: Q1.1 (G), R7.2
- new net: LED20.A, LED21.A, R20.2
- new net: D106.2 (DOUT), D107.4 (DIN)
- new net: D105.2 (DOUT), D106.4 (DIN)
- new net: LED35.A, R34.2
- new net: D108.2 (DOUT), D109.4 (DIN)
- new net: D107.2 (DOUT), D108.4 (DIN)
- new net: LED24.A, R23.2
- new net: LED23.A, R22.2
- new net: LED39.A, R38.2
- new net: D98.2 (DOUT), D99.4 (DIN)
- new net: D97.2 (DOUT), D98.4 (DIN)
- new net: LED14.A, LED15.A, R17.2
- new net: LED31.A, R30.2
- new net: LED25.A, R24.2
- new net: LED42.A, R40.2
- new net: LED2.A, R9.2
- new net: D104.2 (DOUT), D105.4 (DIN)
- new net: LED32.A, R31.2
- new net: LED11.A, R14.2
- new net: D95.2 (DOUT), D96.4 (DIN)
- new net: D100.4 (DIN), D99.2 (DOUT)
- new net: LED33.A, R32.2
- new net: LED29.A, R28.2
- new net: D100.2 (DOUT), D101.4 (DIN)
- new net: LED38.A, R37.2
- new net: D96.2 (DOUT), D97.4 (DIN)
- new net: LED37.A, R36.2
- new net: LED13.A, R16.2
- new net: D101.2 (DOUT), D102.4 (DIN)
- new net CAPS_INDICATOR: U2.19 (PB1)
- new net LED_PWM: R6.1, R7.1, U2.16 (PA6)
- new net PA9: R4.2, U2.30 (PA9)
- new net PB2/BOOT1: U2.20 (PB2), X1.6 (Pin_6)
- new net XTAL_IN: C9.1, U2.5 (PH0_OSCIN), Y1.3
- new net XTAL_OUT: C8.1, U2.6 (PH1_OSCOUT), Y1.1
Other:
- note added: "(*) "Spooky pins": on STM32F4x1, pins A9 and B2 cannot be used for switch matrix: - A9 is meant to be used as a VBUS sensing. It has a undocumented internal pulldown resistor; - B2 is used as BOOT1 during bootup, so it needs an external pulldown for successful bootup"
- note added: "(**) PA9 jumper: a solderable jumper used to tie PA9 to VBUS. It is disconnected by default, hence PA9 is left floating"
- note added: "EEPROM"
- note added: "Spooky pin (*)"
- note added: "USB REMOVAL MOUSEBITES"
- moved on the sheet: C13, C14, C15, C16, C17, C18, D1, D10, D11, D12, D13, D14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

Commit message: Routing work
Parts:
- removed C35: 100n, Capacitor_SMD:C_0805_2012Metric, symbol Device:C_Small
- removed D100, D101, D102, D103, D104, D105, D106, D107, D108, D109, D110, D111, D96, D97, D98, D99: WS2812C, acheron_Components:LED_WS2812B_5.0x5.0mm_P3.2mm, symbol LED:WS2812B
- added C19, C36, C37, C38, C39, C40, C41, C42, C43, C44, C45, C46, C47, C48, C49, C50, C51, C52: 100n, Capacitor_SMD:C_0805_2012Metric, symbol Device:C_Small
- added D100, D112, D113, D114, D115, D116, D117, D118, D119, D120, D121, D122, D123, D124, D125, D126, D127, D128, D95, D96, D97, D98, D99: WS2812C-2020, acheron_Components:LED_WS2812_2020, symbol acheron_Symbols:WS2812B-2020
- added D101, D102, D103, D104, D105, D106, D107, D108, D109, D110: WS2812C-2020, acheron_Components:LED_WS2812_2020_uparrow, symbol acheron_Symbols:WS2812B-2020
- added LED100, LED101, LED102, LED103, LED104, LED105, LED106, LED107, LED108, LED109, LED110, LED111, LED45, LED46, LED47, LED48, LED49, LED50, LED51, LED52, LED53, LED54, LED55, LED56, LED57, LED58, LED59, LED60, LED61, LED62, LED63, LED64, LED65, LED66, LED67, LED68, LED69, LED70, LED71, LED72, LED73, LED74, LED75, LED76, LED77, LED78, LED79, LED80, LED81, LED82, LED83, LED84, LED85, LED86, LED87, LED88, LED89, LED90, LED91, LED92, LED93, LED94, LED95, LED96, LED97, LED98, LED99: LED, acheron_Components:LED_THT_2.54mm, symbol acheron_Symbols:LED
- added R100, R101, R102, R103, R104, R105, R106, R107, R108, R109, R51, R52, R53, R54, R55, R56, R57, R58, R59, R60, R61, R62, R63, R64, R65, R66, R67, R68, R69, R70, R71, R72, R73, R74, R75, R76, R77, R78, R79, R80, R81, R82, R83, R84, R85, R86, R87, R88, R89, R90, R91, R92, R93, R94, R95, R96, R97, R98, R99: 470, Resistor_SMD:R_0805_2012Metric, symbol Device:R_Small
- added R13: 10k, Resistor_SMD:R_0805_2012Metric, symbol Device:R_Small
- D111: renamed from D95; value WS2812C -> WS2812C-2020; footprint acheron_Components:LED_WS2812B_5.0x5.0mm_P3.2mm -> acheron_Components:LED_WS2812_2020; symbol LED:WS2812B -> acheron_Symbols:WS2812B-2020; Manufacturer Part Number LCSC C114587 -> LCSC C965556 (https://www.lcsc.com/product-detail/Light-Emi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; Package 5050 -> 2020; Vendor Part Number WS2812C -> WS2812C-2020
- H1: footprint acheron_MountingHoles:MountingHole_2.5x4.0mm -> MountingHole:MountingHole_2.5mm_Pad
- R5: footprint apollo87h_kicad_library:R_0805_2012Metric -> Resistor_SMD:R_0805_2012Metric
- renumbered C19 to C35, Q2 to Q1, Q1 to Q2, R47 to R10, R48 to R11, R49 to R12, R6 to R14, R7 to R15, R8 to R16, R9 to R17, R10 to R18, R11 to R19, R12 to R20, R13 to R21, R14 to R22, R15 to R23, R16 to R24, R17 to R25, R18 to R26, R19 to R27, R20 to R28, R21 to R29, R22 to R30, R23 to R31, R24 to R32, R25 to R33, R26 to R34, R27 to R35, R28 to R36, R29 to R37, R30 to R38, R31 to R39, R32 to R40, R33 to R41, R34 to R42, R35 to R43, R36 to R44, R37 to R45, R38 to R46, R39 to R47, R40 to R48, R41 to R49, R42 to R50, R43 to R6, R44 to R7, R45 to R8, R46 to R9
Connections:
- net 5V: now also C20.1, D111.4 (VDD), C19.1, C36.1, C37.1, C38.1, C39.1, C40.1, C41.1, C42.1, C43.1, C44.1, C45.1, C46.1, C47.1, C48.1, C49.1, C50.1, C51.1, C52.1, D100.4 (VDD), D101.4 (VDD), D102.4 (VDD), D103.4 (VDD), D104.4 (VDD), D105.4 (VDD), D106.4 (VDD), D107.4 (VDD), D108.4 (VDD), D109.4 (VDD), D110.4 (VDD), D112.4 (VDD), D113.4 (VDD), D114.4 (VDD), D115.4 (VDD), D116.4 (VDD), D117.4 (VDD), D118.4 (VDD), D119.4 (VDD), D120.4 (VDD), D121.4 (VDD), D122.4 (VDD), D123.4 (VDD), D124.4 (VDD), D125.4 (VDD), D126.4 (VDD), D127.4 (VDD), D128.4 (VDD), D95.4 (VDD), D96.4 (VDD), D97.4 (VDD), D98.4 (VDD), D99.4 (VDD); no longer C20.2, D111.1 (VDD)
- net C0: now also SW94.1; no longer SW94.2
- net C10: now also SW100.1, SW110.1; no longer SW100.2, SW111.2
- net C11: now also SW111.2
- net C6: now also SW98.1; no longer SW98.2
- net C9: now also SW99.1; no longer SW110.2, SW99.2
- net GND: now also C20.2, D111.2 (VSS), C19.2, C36.2, C37.2, C38.2, C39.2, C40.2, C41.2, C42.2, C43.2, C44.2, C45.2, C46.2, C47.2, C48.2, C49.2, C50.2, C51.2, C52.2, D100.2 (VSS), D101.2 (VSS), D102.2 (VSS), D103.2 (VSS), D104.2 (VSS), D105.2 (VSS), D106.2 (VSS), D107.2 (VSS), D108.2 (VSS), D109.2 (VSS), D110.2 (VSS), D112.2 (VSS), D113.2 (VSS), D114.2 (VSS), D115.2 (VSS), D116.2 (VSS), D117.2 (VSS), D118.2 (VSS), D119.2 (VSS), D120.2 (VSS), D121.2 (VSS), D122.2 (VSS), D123.2 (VSS), D124.2 (VSS), D125.2 (VSS), D126.2 (VSS), D127.2 (VSS), D128.2 (VSS), D95.2 (VSS), D96.2 (VSS), D97.2 (VSS), D98.2 (VSS), D99.2 (VSS), LED100.K, LED101.K, LED102.K, LED103.K, LED104.K, LED105.K, LED106.K, LED107.K, LED108.K, LED109.K, LED110.K, LED111.K, LED46.K, LED47.K, LED48.K, LED49.K, LED50.K, LED51.K, LED52.K, LED53.K, LED54.K, LED55.K, LED56.K, LED57.K, LED58.K, LED59.K, LED60.K, LED61.K, LED62.K, LED63.K, LED64.K, LED65.K, LED66.K, LED67.K, LED68.K, LED69.K, LED70.K, LED71.K, LED72.K, LED73.K, LED74.K, LED75.K, LED76.K, LED77.K, LED78.K, LED79.K, LED80.K, LED81.K, LED82.K, LED83.K, LED84.K, LED85.K, LED86.K, LED87.K, LED88.K, LED89.K, LED90.K, LED91.K, LED92.K, LED93.K, LED94.K, LED95.K, LED96.K, LED97.K, LED98.K, LED99.K, R13.2, R67.2; no longer C20.1, D111.3 (VSS)
- net PB2/BOOT1: now also R13.1
- net at Q2.3 (D), R16.1, R17.1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: now also LED45.A, R100.1, R101.1, R102.1, R103.1, R104.1, R105.1, R106.1, R107.1, R108.1, R109.1, R51.1, R52.1, R53.1, R54.1, R55.1, R56.1, R57.1, R58.1, R59.1, R60.1, R61.1, R62.1, R63.1, R64.1, R65.1, R66.1, R68.1, R69.1, R70.1, R71.1, R72.1, R73.1, R74.1, R75.1, R76.1, R77.1, R78.1, R79.1, R80.1, R81.1, R82.1, R83.1, R84.1, R85.1, R86.1, R87.1, R88.1, R89.1, R90.1, R91.1, R92.1, R93.1, R94.1, R95.1, R96.1, R97.1, R98.1, R99.1
- net at D88.2 (A), SW101.1: now also SW111.1
- net at D67.2 (A), SW78.1: now also SW94.2; no longer SW94.1
- net at D85.2 (A), SW109.1: now also SW98.2; no longer SW98.1
- new net: LED75.A, R80.2
- new net: D102.1 (DOUT), D103.3 (DIN)
- new net: D101.1 (DOUT), D102.3 (DIN)
- new net: LED109.A, R107.2
- new net: LED81.A, R86.2
- new net: LED59.A, R64.2
- new net: D117.1 (DOUT), D118.3 (DIN)
- new net: D116.1 (DOUT), D117.3 (DIN)
- new net: LED74.A, R79.2
- new net: LED52.A, R57.2
- new net: D118.1 (DOUT), D119.3 (DIN)
- new net: D104.1 (DOUT), D105.3 (DIN)
- new net: D103.1 (DOUT), D104.3 (DIN)
- new net: LED87.A, R92.2
- new net: LED60.A, R65.2
- new net: LED84.A, R89.2
- new net: LED103.A, LED104.A, R104.2
- new net: LED100.A, LED101.A, R102.2
- new net: LED49.A, R54.2
- new net: LED110.A, R108.2
- new net: LED78.A, R83.2
- new net: LED69.A, R74.2
- new net: LED53.A, R58.2
- new net: LED46.A, R51.2
- new net: D95.1 (DOUT), D96.3 (DIN)
- new net: LED80.A, R85.2
- new net: D107.1 (DOUT), D108.3 (DIN)
- new net: D106.1 (DOUT), D107.3 (DIN)
- new net: LED88.A, R93.2
- new net: D96.1 (DOUT), D97.3 (DIN)
- new net: LED85.A, R90.2
- new net: LED86.A, R91.2
- new net: D86.2 (A), SW99.2
- new net: LED68.A, R73.2
- new net: D105.1 (DOUT), D106.3 (DIN)
- new net: LED83.A, R88.2
- new net: LED102.A, R103.2
- new net: D126.1 (DOUT), D127.3 (DIN)
- new net: D125.1 (DOUT), D126.3 (DIN)
- new net: LED65.A, R70.2
- new net: LED76.A, R81.2
- new net: LED77.A, R82.2
- new net: D87.2 (A), SW100.2, SW110.2
- new net: LED45.K, R67.1
- new net: LED54.A, R59.2
- new net: LED98.A, LED99.A, R101.2
- new net: LED66.A, R71.2
- new net: LED72.A, R77.2
- new net: LED61.A, R66.2
- new net: D108.1 (DOUT), D109.3 (DIN)
- new net: D112.1 (DOUT), D113.3 (DIN)
- new net: D111.1 (DOUT), D112.3 (DIN)
- new net: LED51.A, R56.2
- new net: LED55.A, R60.2
- new net: LED62.A, LED63.A, R68.2
- new net: D123.1 (DOUT), D124.3 (DIN)
- new net: D122.1 (DOUT), D123.3 (DIN)
- new net: LED90.A, R95.2
- new net: LED94.A, LED95.A, R99.2
- new net: LED56.A, R61.2
- new net: LED105.A, LED106.A, R105.2
- new net: LED73.A, R78.2
- new net: LED79.A, R84.2
- new net: LED64.A, R69.2
- new net: D115.1 (DOUT), D116.3 (DIN)
- new net: LED107.A, LED108.A, R106.2
- new net: D124.1 (DOUT), D125.3 (DIN)
- new net: LED67.A, R72.2
- new net: LED89.A, R94.2
- new net: LED71.A, R76.2
- new net: D110.1 (DOUT), D111.3 (DIN)
- new net: D127.1 (DOUT), D128.3 (DIN)
- new net: LED93.A, R98.2
- new net: D98.1 (DOUT), D99.3 (DIN)
- new net: D97.1 (DOUT), D98.3 (DIN)
- new net: LED57.A, R62.2
- new net: LED47.A, R52.2
- new net: LED58.A, R63.2
- new net: LED50.A, R55.2
- new net: LED70.A, R75.2
- new net: LED92.A, R97.2
- new net: LED82.A, R87.2
- new net: LED91.A, R96.2
- new net: D100.1 (DOUT), D101.3 (DIN)
- new net: D100.3 (DIN), D99.1 (DOUT)
- new net: D109.1 (DOUT), D110.3 (DIN)
- new net: LED111.A, R109.2
- new net: LED96.A, LED97.A, R100.2
- new net: D121.1 (DOUT), D122.3 (DIN)
- new net: D120.1 (DOUT), D121.3 (DIN)
- new net: D113.1 (DOUT), D114.3 (DIN)
- new net: D114.1 (DOUT), D115.3 (DIN)
- new net: D119.1 (DOUT), D120.3 (DIN)
- new net: LED48.A, R53.2
Other:
- moved on the sheet: C13, C14, C15, C16, C17, C18, C35, D1, D10, D11, D111, D12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

Commit message: Routing work, USB DB sketch
Parts:
- removed C49: 100n, Capacitor_SMD:C_0805_2012Metric, symbol Device:C_Small
- added C52, C53, C54, C55, C56, C57, C58, C59, C60: 100n, Capacitor_SMD:C_0805_2012Metric, symbol Device:C_Small
- added D128, D129, D130, D131, D132, D133, D134, D135, D136: WS2812C-2020, acheron_Components:LED_WS2812_2020, symbol acheron_Symbols:WS2812B-2020
- added FB2: CBW201209U121T, Inductor_SMD:L_0805_2012Metric, symbol Device:Ferrite_Bead_Small
- added GR2: Grounding sign, acheron_Graphics:Grounding_Sign_3.6x3.2mm, symbol Mechanical:MountingHole
- added H1: DB_RGB_PASSTHROUGH, athena_library:rgb_daughterboard_notch_plated_8x4mm, symbol Mechanical:MountingHole_Pad
- added J4: SM04B-SRSS-TB(LF)(SN), acheron_Connectors:PinHeader_1x4_P2.54mm_Angled, symbol Connector_Generic_MountingPin:Conn_01x04_MountingPin
- added LED62: LED, acheron_Components:LED_THT_2.54mm, symbol acheron_Symbols:LED
- added R67: 470, Resistor_SMD:R_0805_2012Metric, symbol Device:R_Small
- added X2: USB_EXPOSED_PINS, acheron_Connectors:PinHeader_1x4_P2.54mm_Vertical, symbol Connector_Generic:Conn_01x04
- added X4: MountingHole, MountingHole:MountingHole_2.2mm_M2_DIN965_Pad, symbol Mechanical:MountingHole
- renumbered C16 to C15, C17 to C16, C15 to C17, C52 to C19, C51 to C20, C50 to C21, C48 to C22, C47 to C23, C46 to C24, C45 to C25, C44 to C26, C43 to C27, C42 to C28, C41 to C29, C40 to C30, C39 to C31, C38 to C32, C37 to C33, C36 to C34, C34 to C36, C33 to C37, C32 to C38, C31 to C39, C30 to C40, C29 to C41, C28 to C42, C27 to C43, C26 to C44, C25 to C45, C24 to C46, C23 to C47, C22 to C48, C21 to C49, C20 to C50, C19 to C51, D122 to D100, D121 to D101, D120 to D102, D119 to D103, D118 to D104, D117 to D105, D116 to D106, D115 to D107, D114 to D108, D113 to D109, D112 to D110, D110 to D112, D109 to D113, D108 to D114, D107 to D115, D106 to D116, D105 to D117, D104 to D118, D103 to D119, D102 to D120, D101 to D121, D100 to D122, D99 to D123, D98 to D124, D97 to D125, D96 to D126, D95 to D127, D125 to D137, D128 to D95, D127 to D96, D126 to D97, D124 to D98, D123 to D99, LED99 to LED100, LED100 to LED101, LED101 to LED102, LED102 to LED103, LED103 to LED104, LED104 to LED105, LED105 to LED106, LED106 to LED107, LED107 to LED108, LED108 to LED109, LED109 to LED110, LED110 to LED111, LED111 to LED112, LED62 to LED63, LED63 to LED64, LED64 to LED65, LED65 to LED66, LED66 to LED67, LED67 to LED68, LED68 to LED69, LED69 to LED70, LED70 to LED71, LED71 to LED72, LED72 to LED73, LED73 to LED74, LED74 to LED75, LED75 to LED76, LED76 to LED77, LED82 to LED78, LED87 to LED79, LED88 to LED80, LED77 to LED81, LED78 to LED82, LED79 to LED83, LED80 to LED84, LED81 to LED85, LED83 to LED86, LED84 to LED87, LED85 to LED88, LED86 to LED89, LED89 to LED90, LED90 to LED91, LED91 to LED92, LED92 to LED93, LED93 to LED94, LED94 to LED95, LED95 to LED96, LED96 to LED97, LED97 to LED98, LED98 to LED99, R8 to R10, R99 to R100, R100 to R101, R101 to R102, R102 to R103, R103 to R104, R104 to R105, R105 to R106, R106 to R107, R107 to R108, R108 to R109, R109 to R110, R67 to R68, R68 to R69, R69 to R70, R70 to R71, R71 to R72, R72 to R73, R73 to R74, R74 to R75, R75 to R76, R76 to R77, R77 to R78, R78 to R79, R9 to R8, R79 to R80, R80 to R81, R81 to R82, R82 to R83, R83 to R84, R84 to R85, R85 to R86, R86 to R87, R10 to R9, R94 to R92, R95 to R93, R96 to R94, R97 to R95, R98 to R96, R87 to R97, R92 to R98, R93 to R99, H1 to X3
Connections:
- net 5V: now also C52.1, C53.1, C54.1, C55.1, C56.1, C57.1, C58.1, C59.1, C60.1, D128.4 (VDD), D129.4 (VDD), D130.4 (VDD), D131.4 (VDD), D132.4 (VDD), D133.4 (VDD), D134.4 (VDD), D135.4 (VDD), D136.4 (VDD), J4.1 (Pin_1), X2.1 (Pin_1); no longer D137.4 (VDD)
- net C11: now also SW101.1, SW111.1; no longer SW101.2, SW111.2
- net C13: now also SW91.2; no longer SW91.1
- net C15: now also SW104.1; no longer SW104.2
- net C2: now also SW80.2; no longer SW80.1
- net D+: now also X2.3 (Pin_3)
- net D-: now also X2.2 (Pin_2)
- net GND: now also R97.2, R98.2, R99.2, C52.2, C53.2, C54.2, C55.2, C56.2, C57.2, C58.2, C59.2, C60.2, D128.2 (VSS), D129.2 (VSS), D130.2 (VSS), D131.2 (VSS), D132.2 (VSS), D133.2 (VSS), D134.2 (VSS), D135.2 (VSS), D136.2 (VSS), FB2.1, H1.1, J4.2 (Pin_2), J4.4 (Pin_4), J4.MP (MountPin), LED62.K, X2.4 (Pin_4); no longer D137.2 (VSS), LED78.K, LED79.K, LED80.K
- net GNDPWR: no longer X3.1
- net at D120.1 (DOUT): now also D121.3 (DIN); no longer D119.3 (DIN)
- net at D120.3 (DIN): now also D119.1 (DOUT); no longer D121.1 (DOUT)
- net at LED45.A, Q2.3 (D), R100.1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: now also LED78.A, LED79.A, LED80.A, R67.1; no longer R97.1, R98.1, R99.1
- net at D105.1 (DOUT): now also D106.3 (DIN); no longer D104.3 (DIN)
- net at D105.3 (DIN): now also D104.1 (DOUT); no longer D106.1 (DOUT)
- net at D103.3 (DIN): now also D102.1 (DOUT); no longer D104.1 (DOUT)
- net at D91.2 (A): now also SW104.2; no longer SW104.1
- net at D118.1 (DOUT): now also D119.3 (DIN); no longer D117.3 (DIN)
- net at D118.3 (DIN): now also D117.1 (DOUT); no longer D119.1 (DOUT)
- net at D126.3 (DIN): now also D125.1 (DOUT); no longer D127.1 (DOUT)
- net at D127.3 (DIN): now also D126.1 (DOUT)
- net at D115.1 (DOUT): now also D116.3 (DIN); no longer D114.3 (DIN)
- net at D115.3 (DIN): now also D114.1 (DOUT); no longer D116.1 (DOUT)
- net at D125.3 (DIN): now also D124.1 (DOUT); no longer D126.1 (DOUT)
- net at D69.2 (A): now also SW80.1; no longer SW80.2
- net at D97.1 (DOUT): now also D98.3 (DIN); no longer D96.3 (DIN)
- net at D97.3 (DIN): now also D96.1 (DOUT); no longer D137.1 (DOUT)
- net at D113.3 (DIN): now also D112.1 (DOUT); no longer D114.1 (DOUT)
- net at D110.1 (DOUT): now also D111.3 (DIN); no longer D109.3 (DIN)
- net at D110.3 (DIN): now also D109.1 (DOUT); no longer D111.1 (DOUT)
- net at D99.1 (DOUT): now also D100.3 (DIN); no longer D98.3 (DIN)
- net at D99.3 (DIN): now also D98.1 (DOUT); no longer D100.1 (DOUT)
- net at D107.1 (DOUT): now also D108.3 (DIN); no longer D106.3 (DIN)
- net at D137.3 (DIN): no longer D98.1 (DOUT)
- net RGB_5V_MAIN: now reaches D95.3 (DIN)
- net RGB_5V_MAIN: now also U3.4 (B); no longer D96.1 (DOUT)
- net at D80.2 (A): now also SW91.1; no longer SW91.2
- net at D123.3 (DIN): now also D122.1 (DOUT); no longer D124.1 (DOUT)
- net at D124.3 (DIN): now also D123.1 (DOUT); no longer D125.1 (DOUT)
- net at D122.3 (DIN): now also D121.1 (DOUT); no longer D123.1 (DOUT)
- net at D113.1 (DOUT): now also D114.3 (DIN); no longer D112.3 (DIN)
- net at D101.1 (DOUT): now also D102.3 (DIN); no longer D100.3 (DIN)
- net at D101.3 (DIN): now also D100.1 (DOUT); no longer D102.1 (DOUT)
- net at D95.1 (DOUT): now also D96.3 (DIN)
- net at D107.3 (DIN): now also D106.1 (DOUT); no longer D108.1 (DOUT)
- net at D103.1 (DOUT): now also D104.3 (DIN); no longer D102.3 (DIN)
- net RGB_5V renamed RGB_5V_DB
- net RGB_5V_DB: now also D127.1 (DOUT), D128.3 (DIN), J4.3 (Pin_3); no longer U3.4 (B)
- new net: FB2.2, X3.1
- new net: D132.1 (DOUT), D133.3 (DIN)
- new net: D131.1 (DOUT), D132.3 (DIN)
- new net: D133.1 (DOUT), D134.3 (DIN)
- new net: LED79.K, R98.1
- new net: D134.1 (DOUT), D135.3 (DIN)
- new net: D129.1 (DOUT), D130.3 (DIN)
- new net: D128.1 (DOUT), D129.3 (DIN)
- new net: D135.1 (DOUT), D136.3 (DIN)
- new net: LED80.K, R99.1
- new net: D130.1 (DOUT), D131.3 (DIN)
- new net: D116.1 (DOUT), D117.3 (DIN)
- new net: D88.2 (A), SW101.2, SW111.2
- new net: LED62.A, R67.2
- new net: D111.1 (DOUT), D112.3 (DIN)
- new net: LED78.K, R97.1
- new net: D108.1 (DOUT), D109.3 (DIN)
Other:
- moved on the sheet: C19, C20, C21, C22, C23, C24, C25, C26, C27, C28, C29, C30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

Commit message: More routing, DRC and post-routing pending
Parts:
- removed C52, C53, C54, C55, C56, C57, C58, C59, C60: 100n, Capacitor_SMD:C_0805_2012Metric, symbol Device:C_Small
- removed D128, D129, D130, D131, D132, D133, D134, D135, D136, D137: WS2812C-2020, acheron_Components:LED_WS2812_2020, symbol acheron_Symbols:WS2812B-2020
- removed J4: SM04B-SRSS-TB(LF)(SN), acheron_Connectors:PinHeader_1x4_P2.54mm_Angled, symbol Connector_Generic_MountingPin:Conn_01x04_MountingPin
- removed M1, M2: USB removal mousebite, athena_library:usbc_removal_mousebite_0.5mm, symbol Mechanical:MountingHole
- removed M3, M4: USB removal mousebite, athena_library:usbc_removal_mousebite_1mm, symbol Mechanical:MountingHole
- removed X4: MountingHole, MountingHole:MountingHole_2.2mm_M2_DIN965_Pad, symbol Mechanical:MountingHole
- added C15: 1u, acheron_Components:CP_EIA-3216-10_Kemet-I_Pad1.58x1.35mm_HandSolder, symbol Device:CP1
- added D1: SMF6.0A, acheron_Components:D_SOD-123, symbol Device:D_Schottky
- H1: value DB_RGB_PASSTHROUGH -> DB_RGB_PASSTHROUGH_HOLE
- renumbered C15 to C16, C16 to C17, C17 to C18, C18 to C19, C19 to C20, C20 to C21, C21 to C22, C22 to C23, C23 to C24, C24 to C25, C25 to C26, C26 to C27, C27 to C28, C28 to C29, C29 to C30, C30 to C31, C31 to C32, C32 to C33, C33 to C34, C34 to C35, C35 to C36, C36 to C37, C37 to C38, C38 to C39, C39 to C40, C40 to C41, C41 to C42, C42 to C43, C43 to C44, C44 to C45, C45 to C46, C46 to C47, C47 to C48, C48 to C49, C49 to C50, C50 to C51, C51 to C52, D101 to D10, D62 to D100, D63 to D101, D64 to D102, D67 to D103, D68 to D104, D69 to D105, D70 to D106, D71 to D107, D72 to D108, D73 to D109, D102 to D11, D74 to D110, D75 to D111, D76 to D112, D77 to D113, D78 to D114, D79 to D115, D80 to D116, D81 to D117, D82 to D118, D83 to D119, D103 to D12, D84 to D120, D85 to D121, D86 to D122, D87 to D123, D88 to D124, D89 to D125, D90 to D126, D91 to D127, D92 to D128, D104 to D13, D105 to D14, D106 to D15, D107 to D16, D108 to D17, D109 to D18, D110 to D19, D93 to D2, D111 to D20, D112 to D21, D113 to D22, D114 to D23, D115 to D24, D116 to D25, D117 to D26, D118 to D27, D119 to D28, D120 to D29, D94 to D3, D121 to D30, D122 to D31, D123 to D32, D124 to D33, D125 to D34, D126 to D35, D127 to D36, D1 to D37, D2 to D38, D3 to D39, D95 to D4, D4 to D40, D5 to D41, D6 to D42, D7 to D43, D8 to D44, D9 to D45, D10 to D46, D11 to D47, D12 to D48, D13 to D49, D96 to D5, D14 to D50, D15 to D51, D16 to D52, D17 to D53, D18 to D54, D19 to D55, D20 to D56, D21 to D57, D22 to D58, D23 to D59, D97 to D6, D24 to D60, D25 to D61, D26 to D62, D27 to D63, D28 to D64, D29 to D65, D30 to D66, D31 to D67, D32 to D68, D48 to D69, D98 to D7, D49 to D70, D33 to D71, D34 to D72, D35 to D73, D36 to D74, D37 to D75, D38 to D76, D39 to D77, D40 to D78, D41 to D79, D99 to D8, D42 to D80, D43 to D81, D44 to D82, D45 to D83, D46 to D84, D47 to D85, D65 to D86, D66 to D87, D50 to D88, D51 to D89, D100 to D9, D52 to D90, D53 to D91, D54 to D92, D55 to D93, D56 to D94, D57 to D95, D58 to D96, D59 to D97, D60 to D98, D61 to D99, LED22 to LED1, LED7 to LED10, LED8 to LED11, LED9 to LED12, LED10 to LED13, LED11 to LED14, LED12 to LED15, LED13 to LED16, LED14 to LED17, LED15 to LED18, LED16 to LED19, LED23 to LED2, LED17 to LED20, LED18 to LED21, LED19 to LED22, LED20 to LED23, LED21 to LED24, LED24 to LED25, LED42 to LED26, LED43 to LED27, LED44 to LED28, LED26 to LED29, LED25 to LED3, LED27 to LED30, LED28 to LED31, LED29 to LED32, LED30 to LED33, LED31 to LED34, LED32 to LED35, LED33 to LED36, LED34 to LED37, LED35 to LED38, LED36 to LED39, LED1 to LED4, LED37 to LED40, LED38 to LED41, LED39 to LED42, LED40 to LED43, LED41 to LED44, LED59 to LED46, LED60 to LED47, LED61 to LED48, LED46 to LED49, LED2 to LED5, LED47 to LED50, LED48 to LED51, LED49 to LED52, LED50 to LED53, LED51 to LED54, LED52 to LED55, LED53 to LED56, LED54 to LED57, LED55 to LED58, LED56 to LED59, LED3 to LED6, LED57 to LED60, LED58 to LED61, LED68 to LED63, LED72 to LED64, LED73 to LED65, LED74 to LED66, LED77 to LED67, LED63 to LED68, LED64 to LED69, LED4 to LED7, LED65 to LED70, LED66 to LED71, LED67 to LED72, LED69 to LED73, LED70 to LED74, LED71 to LED75, LED75 to LED76, LED76 to LED77, LED81 to LED78, LED82 to LED79, LED5 to LED8, LED85 to LED80, LED78 to LED81, LED86 to LED82, LED87 to LED83, LED88 to LED84, LED89 to LED85, LED79 to LED86, LED80 to LED87, LED90 to LED88, LED92 to LED89, LED6 to LED9, LED93 to LED90, LED83 to LED91, LED84 to LED92, LED91 to LED93, R31 to R29, R29 to R30, R30 to R31, R67 to R64, R64 to R65, R65 to R66, R66 to R67, R74 to R73, R75 to R74, R76 to R75, R80 to R76, R81 to R77, R73 to R78, R77 to R79, R78 to R80, R79 to R81, R85 to R83, R86 to R84, R93 to R85, R96 to R86, R83 to R87, R84 to R88, R87 to R89, R97 to R90, R88 to R91, R90 to R92, R91 to R93, R98 to R94, R99 to R95, R92 to R96, R94 to R97, R95 to R98, R89 to R99, SW113 to SW1, SW9 to SW10, SW99 to SW100, SW100 to SW101, SW101 to SW102, SW102 to SW103, SW103 to SW104, SW104 to SW105, SW105 to SW106, SW106 to SW107, SW107 to SW108, SW108 to SW109, SW10 to SW11, SW109 to SW110, SW110 to SW111, SW111 to SW112, SW112 to SW113, SW11 to SW12, SW12 to SW13, SW13 to SW14, SW14 to SW15, SW15 to SW16, SW16 to SW17, SW17 to SW18, SW18 to SW19, SW1 to SW2, SW19 to SW20, SW20 to SW21, SW21 to SW22, SW22 to SW23, SW23 to SW24, SW24 to SW25, SW25 to SW26, SW26 to SW27, SW27 to SW28, SW28 to SW29, SW2 to SW3, SW29 to SW30, SW30 to SW31, SW31 to SW32, SW32 to SW33, SW33 to SW34, SW34 to SW35, SW35 to SW36, SW36 to SW37, SW37 to SW38, SW38 to SW39, SW3 to SW4, SW39 to SW40, SW40 to SW41, SW57 to SW42, SW58 to SW43, SW41 to SW44, SW42 to SW45, SW43 to SW46, SW44 to SW47, SW45 to SW48, SW46 to SW49, SW4 to SW5, SW47 to SW50, SW48 to SW51, SW49 to SW52, SW50 to SW53, SW51 to SW54, SW52 to SW55, SW53 to SW56, SW54 to SW57, SW55 to SW58, SW56 to SW59, SW5 to SW6, SW74 to SW60, SW75 to SW61, SW59 to SW62, SW60 to SW63, SW61 to SW64, SW62 to SW65, SW63 to SW66, SW64 to SW67, SW65 to SW68, SW66 to SW69, SW6 to SW7, SW67 to SW70, SW68 to SW71, SW69 to SW72, SW70 to SW73, SW71 to SW74, SW72 to SW75, SW73 to SW76, SW76 to SW77, SW77 to SW78, SW78 to SW79, SW7 to SW8, SW79 to SW80, SW80 to SW81, SW81 to SW82, SW82 to SW83, SW83 to SW84, SW84 to SW85, SW85 to SW86, SW86 to SW87, SW87 to SW88, SW88 to SW89, SW8 to SW9, SW89 to SW90, SW90 to SW91, SW91 to SW92, SW92 to SW93, SW93 to SW94, SW94 to SW95, SW95 to SW96, SW96 to SW97, SW97 to SW98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
Connections:
- net 5V: now also C15.1, D1.1 (K)
- net C0: now also U2.29 (PA8)
- net C1: now also U2.27 (PB14)
- net C10: now also U2.11 (PA1)
- net C11: now also U2.10 (PA0-WKUP)
- net C12: now also U2.4 (PC15_OSC32OUT)
- net C13: now also U2.17 (PA7)
- net C14: now also U2.40 (PB4)
- net C15: now also U2.39 (PB3)
- net C16: now also U2.38 (PA15)
- net C2: now also U2.25 (PB12)
- net C3: now also U2.21 (B10)
- net C4: now also U2.19 (PB1)
- net C5: now also U2.18 (PB0)
- net C6: now also U2.15 (PA5)
- net C7: now also U2.14 (PA4)
- net C8: now also U2.13 (PA3)
- net C9: now also U2.12 (PA2)
- net CAPS_INDICATOR: now also LED68.K, LED69.K, U2.31 (PA10); no longer U2.19 (PB1)
- net GND: now also R108.2, R30.2, R31.2, R32.2, R48.2, R49.2, R50.2, R65.2, R66.2, R67.2, R78.2, R79.2, R80.2, R81.2, R82.2, R86.2, R87.2, R88.2, R89.2, R91.2, R92.2, R93.2, R96.2, R97.2, R98.2, R99.2, C15.2, D1.2 (A); no longer LED1.K, LED110.K, LED2.K, LED26.K, LED27.K, LED28.K, LED3.K, LED46.K, LED47.K, LED48.K, LED63.K, LED64.K, LED65.K, LED66.K, LED67.K, LED68.K, LED69.K, LED78.K, LED79.K, LED80.K, LED82.K, LED83.K, LED84.K, LED85.K, LED88.K, LED89.K, LED90.K, LED94.K
- net R0: now also U2.46 (PB9)
- net R1: now also D69.1 (K), D70.1 (K), U2.2 (PC13)
- net R2: now also D86.1 (K), D87.1 (K), U2.45 (PB8); no longer D69.1 (K), D70.1 (K)
- net R3: now also U2.41 (PB5); no longer D86.1 (K), D87.1 (K)
- net R5: now also U2.3 (PC14_OSC32IN)
- net at LED45.A, LED81.A, LED86.A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: now also LED1.A, LED110.A, LED2.A, LED26.A, LED27.A, LED28.A, LED3.A, LED46.A, LED47.A, LED48.A, LED63.A, LED64.A, LED65.A, LED66.A, LED67.A, LED78.A, LED79.A, LED80.A, LED82.A, LED83.A, LED84.A, LED85.A, LED88.A, LED89.A, LED90.A, LED94.A; no longer R108.1, R30.1, R31.1, R32.1, R48.1, R49.1, R50.1, R65.1, R66.1, R67.1, R78.1, R79.1, R80.1, R81.1, R82.1, R86.1, R87.1, R88.1, R89.1, R91.1, R92.1, R93.1, R96.1, R97.1, R98.1, R99.1
- new net: LED110.K, R108.1
- new net: LED80.K, R89.1
- new net: LED46.K, R65.1
- new net: LED47.K, R66.1
- new net: LED83.K, R99.1
- new net: LED28.K, R50.1
- new net: LED79.K, R88.1
- new net: LED27.K, R49.1
- new net: LED84.K, R92.1
- new net: LED85.K, R93.1
- new net: LED82.K, R91.1
- new net: LED1.K, R30.1
- new net: LED67.K, R82.1
- new net: LED78.K, R87.1
- new net: LED2.K, R31.1
- new net: LED65.K, R80.1
- new net: LED48.K, R67.1
- new net: LED3.K, R32.1
- new net: LED26.K, R48.1
- new net: LED66.K, R81.1
- new net: LED63.K, R78.1
- new net: LED88.K, R96.1
- new net: LED64.K, R79.1
- new net: LED94.K, R86.1
- new net: LED90.K, R98.1
- new net: LED89.K, R97.1
Other:
- note removed: "USB REMOVAL MOUSEBITES"
- moved on the sheet: D100, D101, D102, D103, D104, D105, D106, D107, D108, D109, D110, D111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

Commit message: Added logos, some DRC
Parts:
- added GR3: Athena Letters, athena_library:athena_letters_plated_22x2.7mm, symbol Mechanical:MountingHole
- added GR4: Athena Label, athena_library:athena_letters_pre-alpha_35x5.6, symbol Mechanical:MountingHole
- added GR5: Acheron Logo, acheron_Logos:acheronLong, symbol Mechanical:MountingHole
- R100, R101, R102, R103, R104, R105, R106, R107, R108, R109, R110, R16, R17, R18, R19, R20, R21, R22, R23, R24, R25, R26, R27, R28, R29, R30, R31, R32, R33, R34, R35, R36, R37, R38, R39, R40, R41, R42, R43, R44, R45, R46, R47, R48, R49, R50, R51, R52, R53, R54, R55, R56, R57, R58, R59, R60, R61, R62, R63, R64, R65, R66, R67, R68, R69, R70, R71, R72, R73, R74, R75, R76, R77, R78, R79, R80, R81, R82, R83, R84, R85, R86, R87, R88, R89, R90, R91, R92, R93, R94, R95, R96, R97, R98, R99: value 470 -> 1k
Other:
- moved on the sheet: LED63, LED64, LED65, LED66, LED67, LED68, LED69, LED70, LED71, LED72, LED73, LED74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

Commit message: Add warning signs, DRC ran, errors fixed
Parts:
- added GR6, GR7, GR8: Warning, acheron_Graphics:Warning_Sign_3.6x3.2mm, symbol Mechanical:MountingHole
Other:
- moved on the sheet: LED1, LED10, LED100, LED101, LED102, LED103, LED104, LED105, LED106, LED107, LED108, LED109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
