File: kicad_files/athena.kicad_sch (KiCad schematic)
At the start: 541 parts, among them J1 SM04B-SRSS-TB(LF)(SN), J2 TYPE-C-31-M12, J3 SM04B-SRSS-TB(LF)(SN), Q1 DTC123JKAT146, Q2 AO3401A, SW1 K2-1187SQ-A4SW-06, SW10 MX Switch, SW100 MX Switch, SW101 MX Switch, SW102 MX Switch, SW103 MX Switch, SW104 MX Switch, SW105 MX Switch, SW106 MX Switch, SW107 MX Switch, SW108 MX Switch, SW109 MX Switch, SW11 MX Switch, SW110 MX Switch, SW111 MX Switch, SW112 MX Switch, SW113 MX Switch, SW12 MX Switch, SW13 MX Switch, SW14 MX Switch, SW15 MX Switch, SW16 MX Switch, SW17 MX Switch, SW18 MX Switch, SW19 MX Switch, SW2 MX Switch, SW20 MX Switch, SW21 MX Switch, SW22 MX Switch, SW23 MX Switch, SW24 MX Switch, SW25 MX Switch, SW26 MX Switch, SW27 MX Switch, SW28 MX Switch, SW29 MX Switch, SW3 MX Switch, SW30 MX Switch, SW31 MX Switch, SW32 MX Switch, SW33 MX Switch, SW34 MX Switch, SW35 MX Switch, SW36 MX Switch, SW37 MX Switch, SW38 MX Switch, SW39 MX Switch, SW4 MX Switch, SW40 MX Switch, SW41 MX Switch, SW42 MX Switch, SW43 MX Switch, SW44 MX Switch, SW45 MX Switch, SW46 MX Switch, SW47 MX Switch, SW48 MX Switch, SW49 MX Switch, SW5 MX Switch, SW50 MX Switch, SW51 MX Switch, SW52 MX Switch, SW53 MX Switch, SW54 MX Switch, SW55 MX Switch, SW56 MX Switch, SW57 MX Switch, SW58 MX Switch, SW59 MX Switch, SW6 MX Switch, SW60 MX Switch, SW61 MX Switch, SW62 MX Switch, SW63 MX Switch, SW64 MX Switch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

Commit message: MCU circuit topology, QOL updates
- Both RCC resistors for USB are now in the bottom layer
- DRC ran again, no errors found
- Changed MCU template to the joker revision 2, meaning removal of some bypass capacitors, adittion of a tantallum 10uF capacitor for VDD and change VCAP pin capacitor to 4.7uF from 2.2uF
Parts:
- removed C12, C5: 4.7u, Capacitor_SMD:C_0402_1005Metric, symbol Device:C_Small
- added C5: 10u, acheron_Components:CP_EIA-3216-10_Kemet-I_Pad1.58x1.35mm_HandSolder, symbol Device:CP1
- C11: value 2.2u -> 4.7u; Specification (none) -> MLCC 10V or more
- C18, C20, C21, C22, C23, C24, C25, C26, C27, C28, C29, C30, C31, C32, C33, C34, C35, C36, C37, C38, C39, C40, C41, C42, C43, C44, C45, C46, C47, C48, C49, C50, C51, C52: Specification MLCC 10V -> MLCC 0805 10V or more
- C8, C9: Specification (none) -> MLCC 10V or more
- D1: Package (none) -> SOD-123; Specification (none) -> Unidirectional TVS 6.0V
- D10, D11, D12, D13, D14, D15, D16, D17, D18, D19, D20, D21, D22, D23, D24, D25, D26, D27, D28, D29, D30, D31, D32, D33, D34, D35, D36, D4, D5, D6, D7, D8, D9: Specification (none) -> Integrated controller serial RGB LED 2020 package
- Q2: Specification (none) -> P-Channel power MOSFET transistor
- U1: Specification (none) -> TSSOP-8 non-volatile 256Kb (32K x 8) I2C EEPROM
- U2: Specification (none) -> 32-bit ARM Cortex-M0+ 128kBytes flash microcontroller
- Y1: Specification (none) -> 8MHz 3225-4P oscillator crystal
Connections:
- net 3V3: now also C5.1
- net GND: now also C5.2
Other:
- note added: "LED BACKLIGHT"
- note added: "RGB UNDERGLOW"
- moved on the sheet: C1, C10, C11, C13, C14, C15, C16, C17, C18, C19, C2, C20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
