File: kicad_files/athena.kicad_sch (KiCad schematic)
At the start: 545 parts, among them J1 Conn_01x02, J2 TYPE-C-31-M12, J3 SM04B-SRSS-TB(LF)(SN), J4 Conn_02x07_Counter_Clockwise, J5 Conn_02x07_Counter_Clockwise, J6 SM04B-SRSS-TB(LF)(SN), Q1 DTC123JKAT146, Q2 AO3401A, Q3 DTC123JKAT146, Q4 DTC123JKAT146, SW1 K2-1187SQ-A4SW-06, SW10 MX Switch, SW100 MX Switch, SW101 MX Switch, SW102 MX Switch, SW103 MX Switch, SW104 MX Switch, SW105 MX Switch, SW106 MX Switch, SW107 MX Switch, SW108 MX Switch, SW109 MX Switch, SW11 MX Switch, SW110 MX Switch, SW111 MX Switch, SW112 MX Switch, SW113 MX Switch, SW12 MX Switch, SW13 MX Switch, SW14 MX Switch, SW15 MX Switch, SW16 MX Switch, SW17 MX Switch, SW18 MX Switch, SW19 MX Switch, SW2 MX Switch, SW20 MX Switch, SW21 MX Switch, SW22 MX Switch, SW23 MX Switch, SW24 MX Switch, SW25 MX Switch, SW26 MX Switch, SW27 MX Switch, SW28 MX Switch, SW29 MX Switch, SW3 MX Switch, SW30 MX Switch, SW31 MX Switch, SW32 MX Switch, SW33 MX Switch, SW34 MX Switch, SW35 MX Switch, SW36 MX Switch, SW37 MX Switch, SW38 MX Switch, SW39 MX Switch, SW4 MX Switch, SW40 MX Switch, SW41 MX Switch, SW42 MX Switch, SW43 MX Switch, SW44 MX Switch, SW45 MX Switch, SW46 MX Switch, SW47 MX Switch, SW48 MX Switch, SW49 MX Switch, SW5 MX Switch, SW50 MX Switch, SW51 MX Switch, SW52 MX Switch, SW53 MX Switch, SW54 MX Switch, SW55 MX Switch, SW56 MX Switch, SW57 MX Switch, SW58 MX Switch, SW59 MX Switch, SW6 MX Switch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

Commit message: Start porting design to JLCPCB-compliant parts
Parts:
- removed D1: RB060M-60TR, acheron_Components:D_SOD-123, symbol Device:D_Schottky
- removed Q1, Q3, Q4: DTC123JKAT146, Package_TO_SOT_SMD:SOT-23, symbol acheronSymbols:DTC123J
- removed U4: MCP1700T-3302E/TT, Package_TO_SOT_SMD:SOT-23, symbol Regulator_Linear:MCP1700-3302E_SOT23
- added C11: 10n, Capacitor_SMD:C_0402_1005Metric, symbol Device:C_Small
- added D2: B5819W-SL, acheron_Components:D_SOD-123, symbol Device:D_Schottky
- added Q1, Q2, Q4, Q5: 2N7002, Package_TO_SOT_SMD:SOT-23, symbol Transistor_FET:2N7002
- added R12, R6: 100R, Resistor_SMD:R_0402_1005Metric, symbol Device:R_Small
- added R13, R33, R5: 10k, Resistor_SMD:R_0402_1005Metric, symbol Device:R_Small
- added R18: 100, Resistor_SMD:R_0402_1005Metric, symbol Device:R_Small
- added R87: 100, Resistor_SMD:R_0805_2012Metric, symbol Device:R_Small
- added R91: 10k, Resistor_SMD:R_0805_2012Metric, symbol Device:R_Small
- added U4: SGM2036-3.3YN5G/TR, acheron_Components:SOT-23-5, symbol acheron_Symbols:SGM2036
- C12: renamed from C5; footprint Capacitor_SMD:C_0805_2012Metric -> Capacitor_SMD:C_0402_1005Metric; Package C0805 -> C0402; Specification MLCC 0805 10V or more -> MLCC 10V or more
- C18: renamed from C17; footprint Capacitor_SMD:C_0805_2012Metric -> Capacitor_SMD:C_0402_1005Metric; Package C0805 -> C0402; Specification MLCC 0805 10V or more -> MLCC 0402 10V or more
- C19: renamed from C18; footprint Capacitor_SMD:C_0805_2012Metric -> Capacitor_SMD:C_0402_1005Metric; Package C0805 -> C0402; Specification MLCC 0805 10V or more -> MLCC 0402 10V or more
- C5: renamed from C11; footprint Capacitor_SMD:C_0805_2012Metric -> Capacitor_SMD:C_0402_1005Metric; Package C0805 -> C0402; Specification MLCC 10V -> MLCC 10V or more
- F1: value mSMD110-16V -> nSMD100-16V; footprint Fuse:Fuse_1812_4532Metric -> Fuse:Fuse_1206_3216Metric; Manufacturer Part Number mSMD110-16V -> nSMD100-16V; Package F1812 -> F1206; Specification 1.1A hold, 2.2A trip PTC resettable fuse -> 1A hold, 1.8A trip PTC resettable fuse; Vendor Part Number LCSC C69691 -> LCSC C70082
- FB1, FB2: value CBW201209U121T -> GZ2012D601TF; Manufacturer Guangdong Fenghua Advanced Tech -> Sunlord; Manufacturer Part Number CBW201209U121T -> GZ2012D601TF; Specification 120R @ 100MHz ferrite bead -> 600R @ 100MHz ferrite bead; Vendor Part Number LCSC C139186 -> LCSC C1017
- R10: renamed from R8; footprint Resistor_SMD:R_0805_2012Metric -> Resistor_SMD:R_0402_1005Metric; Package R0805 -> R0402
- R11: renamed from R3; footprint Resistor_SMD:R_0805_2012Metric -> Resistor_SMD:R_0402_1005Metric; Package R0805 -> R0402
- R15: renamed from R11; footprint Resistor_SMD:R_0805_2012Metric -> Resistor_SMD:R_0402_1005Metric; Package R0805 -> R0402
- R16: renamed from R12; footprint Resistor_SMD:R_0805_2012Metric -> Resistor_SMD:R_0402_1005Metric; Package R0805 -> R0402
- R17: renamed from R13; footprint Resistor_SMD:R_0805_2012Metric -> Resistor_SMD:R_0402_1005Metric; Package R0805 -> R0402
- R3: renamed from R7; footprint Resistor_SMD:R_0805_2012Metric -> Resistor_SMD:R_0402_1005Metric; Package R0805 -> R0402
- R4: renamed from R9; footprint Resistor_SMD:R_0805_2012Metric -> Resistor_SMD:R_0402_1005Metric; Package R0805 -> R0402
- R7: renamed from R6; footprint Resistor_SMD:R_0805_2012Metric -> Resistor_SMD:R_0402_1005Metric; Package R0805 -> R0402
- U2: value 24LC256-I/SN -> AT24C256C-SSHL-T; Manufacturer Part Number 24LC256-I/SN -> AT24C256C-SSHL-T; Vendor Part Number LCSC C411625 -> LCSC C6482
- U3: symbol acheronSymbols:STM32F401-LQFP64 -> acheron_Symbols:STM32F401-LQFP64
- U5: value TXS0101DBVR -> TXS0101DRLR; footprint acheron_Components:SOT-23-6 -> acheron_Components:SOT-563; Package SOT-23-6 -> SOT-563; Vendor Part Number LCSC C132604 -> LCSC C131928
- X3: renamed from J4; value Conn_02x07_Counter_Clockwise -> EXTRA_PINS
- X4: renamed from J5; value Conn_02x07_Counter_Clockwise -> EXTRA_PINS
- Y1: value 7325-0800A2010-00 -> TAXM8M4RFDCET2T; Manufacturer XTY -> TAE; Manufacturer Part Number 7325-0800A2010-00 -> TAXM8M4RFDCET2T; Specification 8MHz 3225-4P oscillator crystal -> (none); Vendor Part Number LCSC C389817 (https://lcsc.com/product-detail/Crystals_XTY-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 -> LCSC C403948
- renumbered C12 to C13, C13 to C14, C14 to C15, C15 to C16, C16 to C17, C19 to C20, C20 to C21, C21 to C22, C22 to C23, C23 to C24, C24 to C25, C25 to C26, C26 to C27, C27 to C28, C28 to C29, C29 to C30, C30 to C31, C31 to C32, C32 to C33, C33 to C34, C34 to C35, C35 to C36, C36 to C37, C37 to C38, C38 to C39, C39 to C40, C40 to C41, C41 to C42, C42 to C43, C43 to C44, C44 to C45, C45 to C46, C46 to C47, C47 to C48, C48 to C49, C49 to C50, C50 to C51, C51 to C52, C52 to C53, D2 to D1, J6 to J4, Q2 to Q3, R92 to R100, R93 to R101, R94 to R102, R95 to R103, R96 to R104, R97 to R105, R98 to R106, R99 to R107, R100 to R108, R101 to R109, R102 to R110, R103 to R111, R104 to R112, R105 to R113, R106 to R114, R107 to R115, R108 to R116, R10 to R14, R14 to R19, R15 to R20, R16 to R21, R17 to R22, R18 to R23, R19 to R24, R20 to R25, R21 to R26, R22 to R27, R23 to R28, R24 to R29, R25 to R30, R26 to R31, R27 to R32, R28 to R34, R29 to R35, R30 to R36, R31 to R37, R32 to R38, R33 to R39, R34 to R40, R35 to R41, R36 to R42, R37 to R43, R38 to R44, R39 to R45, R40 to R46, R41 to R47, R42 to R48, R43 to R49, R44 to R50, R45 to R51, R46 to R52, R47 to R53, R48 to R54, R49 to R55, R50 to R56, R51 to R57, R52 to R58, R53 to R59, R54 to R60, R55 to R61, R56 to R62, R57 to R63, R58 to R64, R59 to R65, R60 to R66, R61 to R67, R62 to R68, R63 to R69, R64 to R70, R65 to R71, R66 to R72, R67 to R73, R68 to R74, R69 to R75, R70 to R76, R71 to R77, R72 to R78, R73 to R79, R4 to R8, R74 to R80, R75 to R81, R76 to R82, R77 to R83, R78 to R84, R79 to R85, R80 to R86, R81 to R88, R82 to R89, R5 to R9, R83 to R90, R84 to R92, R85 to R93, R86 to R94, R87 to R95, R88 to R96, R89 to R97, R90 to R98, R91 to R99, X3 to X5, X4 to X6
Connections:
- net 3V3: now also D2.2 (A), U4.5 (OUT)
- net 5V: now also D2.1 (K), U4.1 (IN), U4.3 (EN)
- net BOOT0: now also R5.2
- net CAPS_INDICATOR: now also R87.1
- net GND: now also FB2.2, C11.1, Q1.2 (S), Q2.2 (S), Q4.2 (S), Q5.2 (S), R13.1, R33.1, R91.1, U4.2 (GND); no longer FB2.1
- net LED_PWM: now also R18.1
- net at X5.1: now also FB2.1; no longer FB2.2
- net at D1.2 (A), SW1.2 (B): now also R12.2
- net at R16.1, R17.1: now also Q4.3 (D)
- net at LED68.K, LED69.K: now also Q5.3 (D)
- net at R11.1: now also Q2.3 (D), R6.1
- new net: Q1.3 (D), R5.1
- new net: Q4.1 (G), R18.2, R33.2
- new net: Q2.1 (G), R12.1, R13.2
- new net: C11.2, U4.4 (BP/FB)
- new net: Q1.1 (G), R6.2
- new net: Q5.1 (G), R87.2, R91.2
Other:
- moved on the sheet: C12, C5, C7, C8, D1, F1, LED1, LED10, LED100, LED101, LED102, LED103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

Commit message: Corrections for some DRC issues
Parts:
- removed C20: 1u, acheron_Components:CP_EIA-3216-10_Kemet-I_Pad1.58x1.35mm_HandSolder, symbol Device:CP1
- added C20: 1u, Capacitor_SMD:C_0805_2012Metric, symbol Device:C
- added GR6: Warning, acheron_Graphics:Warning_Sign_3.6x3.2mm, symbol Mechanical:MountingHole
- added R3: 1.5k, Resistor_SMD:R_0402_1005Metric, symbol Device:R_Small
- D3: Manufacturer (none) -> SUNMATE Elec; Manufacturer Part Number (none) -> SMF6.0A; Package SOD-123 -> SOD-123FL; Vendor Part Number (none) -> LCSC C399281
- renumbered C9 to C10, C10 to C11, C11 to C12, C12 to C7, C7 to C8, C8 to C9, GR6 to GR7, GR7 to GR8, GR8 to GR9, LED9 to LED10, LED10 to LED11, LED11 to LED12, LED12 to LED13, LED13 to LED14, LED14 to LED15, LED15 to LED16, LED16 to LED17, LED17 to LED18, LED18 to LED19, LED19 to LED20, LED20 to LED21, LED21 to LED22, LED22 to LED23, LED23 to LED24, LED24 to LED25, LED25 to LED3, LED3 to LED4, LED4 to LED5, LED5 to LED6, LED6 to LED7, LED7 to LED8, LED8 to LED9, R7 to R10, R99 to R100, R100 to R101, R101 to R102, R102 to R103, R103 to R104, R104 to R105, R105 to R106, R106 to R107, R107 to R108, R108 to R109, R8 to R11, R109 to R110, R110 to R111, R111 to R112, R112 to R113, R113 to R114, R114 to R115, R115 to R116, R116 to R117, R9 to R12, R10 to R14, R14 to R15, R15 to R16, R16 to R17, R17 to R18, R18 to R19, R19 to R20, R20 to R21, R21 to R22, R22 to R23, R23 to R24, R24 to R25, R25 to R26, R26 to R27, R27 to R28, R28 to R29, R29 to R30, R30 to R31, R31 to R32, R32 to R37, R37 to R38, R38 to R39, R3 to R4, R39 to R40, R40 to R41, R41 to R42, R42 to R43, R43 to R44, R44 to R45, R45 to R46, R46 to R47, R47 to R48, R48 to R49, R4 to R5, R49 to R50, R50 to R51, R51 to R52, R52 to R53, R53 to R54, R54 to R55, R55 to R56, R56 to R57, R57 to R58, R58 to R59, R5 to R6, R59 to R60, R60 to R61, R61 to R62, R62 to R63, R63 to R64, R64 to R65, R65 to R66, R66 to R67, R67 to R68, R68 to R69, R6 to R7, R69 to R70, R70 to R71, R71 to R72, R72 to R73, R73 to R74, R74 to R75, R75 to R76, R76 to R77, R77 to R78, R78 to R79, R11 to R8, R79 to R80, R80 to R81, R81 to R82, R82 to R83, R83 to R84, R84 to R85, R85 to R86, R86 to R87, R87 to R88, R88 to R89, R12 to R9, R89 to R90, R90 to R91, R91 to R92, R92 to R93, R93 to R94, R94 to R95, R95 to R96, R96 to R97, R97 to R98, R98 to R99
Connections:
- net 3V3: now also R3.2
- net 5V: now also C20.1
- net D+: now also R3.1
- net GND: now also R14.2, R37.2, C20.2; no longer LED3.K, R14.1
- net at J2.B5 (CC2): now also R14.1; no longer R14.2
- net at LED1.A, LED2.A, LED26.A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: now also LED3.A; no longer R37.1
- new net: LED3.K, R37.1
Other:
- moved on the sheet: LED3, R14, R37

Commit message: More DRC corrections
Parts:
- U5: value TXS0101DRLR -> TXS0101DBVR; footprint acheron_Components:SOT-563 -> acheron_Components:SOT-23-6; Package SOT-563 -> SOT-23; Vendor Part Number LCSC C131928 -> LCSC C132604
Changed lines of the file:
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@@
     (title "Athena PCB schematic")
     (date "2022-01-28")
-    (rev "V2.1.0")
+    (rev "V2.1.1")
     (company "Acheron Project")
     (comment 1 "Designed by Gondolindrim")
@@
     (in_bom yes) (on_board yes)
     (property "Reference" "U5" (id 0) (at 601.98 262.255 0))
-    (property "Value" "TXS0101DRLR" (id 1) (at 601.98 264.795 0)
+    (property "Value" "TXS0101DBVR" (id 1) (at 601.98 264.795 0)
       (effects (font (size 0.762 0.762)))
     )
-    (property "Footprint" "acheron_Components:SOT-563" (id 2) (at 601.98 263.525 0)
+    (property "Footprint" "acheron_Components:SOT-23-6" (id 2) (at 601.98 263.525 0)
       (effects (font (size 1.27 1.27)) hide)
     )
@@
       (effects (font (size 1.27 1.27)) hide)
     )
-    (property "Package" "SOT-563" (id 7) (at 601.98 263.525 0)
+    (property "Package" "SOT-23" (id 7) (at 601.98 263.525 0)
       (effects (font (size 1.27 1.27)) hide)
     )
@@
       (effects (font (size 1.27 1.27)) hide)
     )
-    (property "Vendor Part Number" "LCSC C131928" (id 10) (at 601.98 263.525 0)
+    (property "Vendor Part Number" "LCSC C132604" (id 10) (at 601.98 263.525 0)
       (effects (font (size 1.27 1.27)) hide)
     )
@@
     )
     (path "/6f556440-bf01-4dc9-bfef-0ee4385d954a"
-      (reference "U5") (unit 1) (value "TXS0101DRLR") (footprint "acheron_Components:SOT-563")
+      (reference "U5") (unit 1) (value "TXS0101DBVR") (footprint "acheron_Components:SOT-23-6")
     )
     (path "/4013434a-d80b-495e-97c4-53e000bb1df9"

Commit message: Add metadata to components
Parts:
- C1, C15, C16, C3, C4, C7: Manufacturer (none) -> Samsung; Manufacturer Part Number (none) -> CL05B104KB54PNC; Specification MLCC 10V or more -> 50V 100nF X7R ±10% 0402 MLCC; Vendor Part Number (none) -> LCSC C307331
- C10, C11: value 16p -> 15p; Manufacturer (none) -> Guangdong Fenghua Advanced Tech; Manufacturer Part Number (none) -> 0402CG150J500NT; Specification MLCC 10V or more -> 50V 15pF C0G ±5% 0402 MLCC; Vendor Part Number (none) -> LCSC C1548
- C12: Manufacturer (none) -> Samsung; Manufacturer Part Number (none) -> CL05B103KB5NNNC; Specification MLCC 10V -> 50V 10nF X7R ±10% 0402 MLCC; Vendor Part Number (none) -> LCSC C15195
- C13, C17: Manufacturer (none) -> Samsung; Manufacturer Part Number (none) -> CL05A475MP5NRNC; Specification MLCC 10V or more -> 10V 4.7uF X5R ±20% 0402 MLCC; Vendor Part Number (none) -> LCSC C23733
- C14: Manufacturer (none) -> Samsung; Manufacturer Part Number (none) -> CL05B103KB5NNNC; Specification MLCC 10V or more -> 50V 10nF X7R ±10% 0402 MLCC; Vendor Part Number (none) -> LCSC C15195
- C18, C19: Manufacturer (none) -> Samsung; Manufacturer Part Number (none) -> CL05B104KB54PNC; Specification MLCC 0402 10V or more -> 50V 100nF X7R ±10% 0402 MLCC; Vendor Part Number (none) -> LCSC C307331
- C2: Manufacturer (none) -> Samsung; Manufacturer Part Number (none) -> CL05B104KB54PNC; Specification (none) -> 50V 100nF X7R ±10% 0402 MLCC; Vendor Part Number (none) -> LCSC C307331
- C20, C8, C9: Manufacturer (none) -> Guangdong Fenghua Advanced Tech; Manufacturer Part Number (none) -> 0805B105K500NT; Specification MLCC 10V -> 50V 1uF X7R ±10% 0805 MLCC; Vendor Part Number (none) -> LCSC C215803
- C21, C22, C23, C24, C25, C26, C27, C28, C29, C30, C31, C32, C33, C34, C35, C36, C37, C38, C39, C40, C41, C42, C43, C44, C45, C46, C47, C48, C49, C50, C51, C52, C53: Manufacturer (none) -> Samsung; Manufacturer Part Number (none) -> CL21B104KCFNNNE; Specification MLCC 0805 10V or more -> 100V 100nF X7R ±10% 0805 MLCC; Vendor Part Number (none) -> LCSC C28233
- C5: Manufacturer (none) -> Samsung; Manufacturer Part Number (none) -> CL05A106MQ5NUNC; Specification MLCC 10V or more -> 6.3V 10uF X5R ±20% 0402 MLCC; Vendor Part Number (none) -> LCSC C15525
- C6: Manufacturer (none) -> AVX; Manufacturer Part Number (none) -> TAJA106K016RNJ; Specification Tantallum 10V -> 16V 1uF Tantallum; Vendor Part Number (none) -> LCSC C7171
- D1, D100, D101, D102, D103, D104, D105, D106, D107, D108, D109, D110, D111, D112, D113, D114, D115, D116, D117, D118, D119, D120, D121, D122, D123, D124, D125, D126, D127, D128, D37, D38, D39, D40, D41, D42, D43, D44, D45, D46, D47, D48, D49, D50, D51, D52, D53, D54, D55, D56, D57, D58, D59, D60, D61, D62, D63, D64, D65, D66, D67, D68, D69, D70, D71, D72, D73, D74, D75, D76, D77, D78, D79, D80, D81, D82, D83, D84, D85, D86, D87, D88, D89, D90, D91, D92, D93, D94, D95, D96, D97, D98, D99: Manufacturer (none) -> Semtech; Manufacturer Part Number (none) -> 1N4148W; Vendor Part Number (none) -> LCSC C81598
- Q1, Q2, Q4, Q5: Manufacturer (none) -> Changjiang Electronics Tech; Manufacturer Part Number (none) -> 2N7002; Package (none) -> SOT-23; Specification (none) -> N-channel signal MOSFET transistor; Vendor Part Number (none) -> LCSC C8545
- Q3: Specification P-Channel power MOSFET transistor -> P-channel power MOSFET transistor
- R1, R2: Manufacturer (none) -> Uniroyal; Manufacturer Part Number (none) -> 0402WGF4701TCE; Specification (none) -> ±1% 1/16W Thick Film Resistors 50V 0402
- R10, R14: Manufacturer (none) -> Uniroyal; Manufacturer Part Number (none) -> 0402WGF5101TCE; Specification (none) -> ±1% 1/16W Thick Film Resistors 50V 0805
- R100, R101, R102, R103, R104, R105, R106, R107, R108, R109, R110, R111, R112, R113, R114, R115, R116, R117, R20, R21, R22, R23, R24, R25, R26, R27, R28, R29, R30, R31, R32, R34, R35, R36, R37, R38, R39, R40, R41, R42, R43, R44, R45, R46, R47, R48, R49, R50, R51, R52, R53, R54, R55, R56, R57, R58, R59, R60, R61, R62, R63, R64, R65, R66, R67, R68, R69, R70, R71, R72, R73, R74, R75, R76, R77, R78, R79, R80, R81, R82, R83, R84, R85, R86, R87, R89, R90, R91, R93, R94, R95, R96, R97, R98, R99: Manufacturer (none) -> Uniroyal; Manufacturer Part Number (none) -> 0805W8F1001T5E; Specification (none) -> ±1% 125mW Thick Film Resistors 150V 0805
- R11, R12: Manufacturer (none) -> Uniroyal; Manufacturer Part Number (none) -> 0805W8F1003T5E; Specification (none) -> ±1% 125mW Thick Film R0805 Resistors; Vendor Part Number (none) -> LCSC C149504
- R13, R16, R17, R33, R6: Manufacturer (none) -> Uniroyal; Manufacturer Part Number (none) -> 0402WGF1002TCE; Specification (none) -> ±1% 1/16W Thick Film Resistors 50V 0402; Vendor Part Number (none) -> LCSC C25744
- R15, R92: Manufacturer (none) -> Uniroyal; Manufacturer Part Number (none) -> 0402WGF1002TCE; Package R0805 -> R0402; Specification (none) -> ±1% 1/16W Thick Film Resistors 50V 0402; Vendor Part Number (none) -> LCSC C25744
- R18, R19, R7, R8, R9: Manufacturer (none) -> Uniroyal; Manufacturer Part Number (none) -> 0402WGF1000TCE; Specification (none) -> ±1% 1/16W Thick Film Resistors 50V 0402; Vendor Part Number (none) -> LCSC C25076
- R3: Manufacturer (none) -> Uniroyal; Manufacturer Part Number (none) -> 0402WGF1501TCE; Specification (none) -> ±1% 1/16W Thick Film Resistors 50V 0402
- R4: Manufacturer (none) -> Uniroyal; Manufacturer Part Number (none) -> 0402WGF3303TCE; Specification (none) -> ±1% 1/16W Thick Film Resistors 50V 0402; Vendor Part Number (none) -> LCSC C25778
- R5: Manufacturer (none) -> Uniroyal; Manufacturer Part Number (none) -> 0402WGF1004TCE; Specification (none) -> ±1% 1/16W Thick Film Resistors 50V 0402
- R88: Manufacturer (none) -> Uniroyal; Manufacturer Part Number (none) -> 0402WGF1000TCE; Package R0805 -> R0402; Specification (none) -> ±1% 1/16W Thick Film Resistors 50V 0402; Vendor Part Number (none) -> LCSC C25076
- SW1: Specification Surface-mounted SPST tactile push button -> 5.2mm 1.5mm Round Button SPST
- U4: value SGM2036-3.3YN5G/TR -> SGM2007-3.3XN5/TR; Manufacturer Part Number SGM2036-3.3YN5G/TR -> SGM2007-3.3XN5/TR; Specification (none) -> Fixed 5.5V 3.3V 300mV @ 300mA SOT-23-5 Low Dropout Regulator; Vendor Part Number LCSC C92402 -> LCSC C193687
- X?: renamed from J1; now left out of the parts list
- Y1: Package Y_3225_4P -> Y3225_4P; Specification (none) -> 8MHz 3225-4P oscillator crystal
- renumbered J2 to J1

Commit message: DRC corrections, metadata add
- Added LCSC number for missing components
- DRC corrections: diodes courtyard overlaps
Parts:
- Q3: Manufacturer Part Number BORN -> Alpha & Omega Semicon; Vendor Part Number LCSC C306862 -> LCSC C15127
- R1, R2: Vendor Part Number (none) -> LCSC C25900
- R10, R14: Vendor Part Number (none) -> LCSC C25905
- R100, R101, R102, R103, R104, R105, R106, R107, R108, R109, R110, R111, R112, R113, R114, R115, R116, R117, R20, R21, R22, R23, R24, R25, R26, R27, R28, R29, R30, R31, R32, R34, R35, R36, R37, R38, R39, R40, R41, R42, R43, R44, R45, R46, R47, R48, R49, R50, R51, R52, R53, R54, R55, R56, R57, R58, R59, R60, R61, R62, R63, R64, R65, R66, R67, R68, R69, R70, R71, R72, R73, R74, R75, R76, R77, R78, R79, R80, R81, R82, R83, R84, R85, R86, R87, R89, R90, R91, R93, R94, R95, R96, R97, R98, R99: Vendor Part Number (none) -> LCSC C17513
- R3: Vendor Part Number (none) -> LCSC C25867
- R5: Vendor Part Number (none) -> LCSC C26083
- gave numbers to parts that had none: 1
- renumbered J3 to J2, J4 to J3, X3 to X4, X4 to X5, X5 to X6, X6 to X7

Commit message: Edit component metadata
Parts:
- U3: Manufacturer Part Number STM32F401RBT6 -> STM32F401RCT6; Vendor Part Number LCSC C75278 -> LCSC C74524
Changed lines of the file:
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@@
     (title "Athena PCB schematic")
     (date "2022-01-29")
-    (rev "V2.1.3")
+    (rev "V2.1.4")
     (company "Acheron Project")
     (comment 1 "Designed by Gondolindrim")
@@
       (effects (font (size 1.27 1.27)) hide)
     )
-    (property "Manufacturer Part Number" "STM32F401RBT6" (id 5) (at 259.08 100.33 0)
+    (property "Manufacturer Part Number" "STM32F401RCT6" (id 5) (at 259.08 100.33 0)
       (effects (font (size 1.27 1.27)) hide)
     )
@@
       (effects (font (size 1.27 1.27)) hide)
     )
-    (property "Vendor Part Number" "LCSC C75278" (id 9) (at 259.08 100.33 0)
+    (property "Vendor Part Number" "LCSC C74524" (id 9) (at 259.08 100.33 0)
       (effects (font (size 1.27 1.27)) hide)
     )
